File: hardware/gameflopMB_1/gameflopMB_1.kicad_sch (KiCad schematic)
At the start: 2 parts, among them IC1 MAX7219CNG, IC2 STM32G431RBT6

Commit message: commit
Parts:
- added D1: LED, symbol Device:LED
- added J1: Jack-DC, symbol Connector:Jack-DC
- added J2: USB_B_Micro, symbol Connector:USB_B_Micro
- added J3: Micro_SD_Card, symbol Connector:Micro_SD_Card
- added J4: Conn_01x02_Pin, symbol Connector:Conn_01x02_Pin
- added U1: TP4056, Package_SO:SOIC-8-1EP_3.9x4.9mm_P1.27mm_EP2.29x3mm, symbol tp4056:TP4056
- added U2: TPS613222ADBV, Package_TO_SOT_SMD:SOT-23-5, symbol Regulator_Switching:TPS613222ADBV
